File: Images/OmniBot-Joystick-Schematic/OmniBot-Joystick-Schematic.sch (KiCad schematic (older format))
At the start: 12 parts

Commit message: Updated schematic
Parts:
- removed R, R? (x3): 220 OHM RESISTOR, 0603, symbol SparkFun-Resistors:220KOHM-0603-1_10W-1%
Connections:
- net +5V: no longer j.2 (PIN2), j?.2 (PIN2), j?.2 (PIN2), j?.2 (PIN2)
- net 3.3V: now also j.2 (PIN2), j?.2 (PIN2), j?.2 (PIN2), j?.2 (PIN2)
- net BUTTON_1: now also j.1 (PIN1); no longer j.4 (PIN3)
- net BUTTON_2: now also j?.1 (PIN1); no longer j?.4 (PIN3)
- net BUTTON_3: now also j?.1 (PIN1); no longer j?.4 (PIN3)
- net BUTTON_4: now also j?.1 (PIN1); no longer j?.4 (PIN3)
Other:
- note added: "Note: Resistors not needed as Arduino has internal \npullup resistors. Also, it does not matter which set \nof pins used, only matters the pins are beside \neachother."
